File: Arduino/PCB/TempSensor/TempSensor.sch (EAGLE design)
At the start: 13 parts, among them IC1 DS18B20, U1 ATMEGA328-AU, X1 16Mhz

Commit message: sensor pcb
Parts:
- removed JP2, JP3: (no value), jumper:JP1E
- added C3: 100n, rcl:C-EUC0805
- added J1, J2: FTDI_DEVICE, SparkFun-Connectors:FTDI_DEVICE
- added JP6: (no value), jumper:JP1E
- added JP7, JP8: (no value), jumper:JP2E
- added LED1: 2mA, led:LED3MM
- added R2: 580, rcl:R-EU_R0603
- added R3: 10k, rcl:R-EU_R0805
- added SJ2: (no value), jumper:SJ2W
- added U$3: IE0503D, xp_power:IE0503D
- JP1: device jumper:JP1E -> jumper:JP2E
- R1: value (none) -> 4k7
Connections:
- removed net N$3: JP3.2, XB1.VCC
- new net +5V: J1.VCC, JP1.1
- new net N$11: JP6.2, U$3.+VIN
- new net N$14: JP6.1, U$3.-VIN
- new net N$15: LED1.C, R2.2
- new net N$16: R2.1, U1.(PCINT22/OC0A/AIN0)_PD6
- new net N$17: SJ2.2, U1.(PCINT23/AIN1)_PD7
- new net N$18: JP7.3, XB1.DOUT
- new net N$19: JP8.3, XB1.DIN/!CONFIG
- new net N$20: C3.1, J2.VCC, R3.1, U1.PC6_(!RESET/PCINT14)
- new net N$21: C3.2, J1.DTR
- new net N$22: J2.RXI, U1.(PCINT3/OC2A/MOSI)_PB3
- new net N$23: J2.DTR, U1.PB5_(SCK/PCINT5)
- new net N$24: J2.TXO, U1.(PCINT4/MISO)_PB4
- new net VCC: J2.CTS, JP1.2, LED1.A, SJ2.1, U$2.VCC, U1.AVCC, U1.VCC, U1.VCC_2
- net +3V3: now also JP1.3, R3.2, U$3.+VOUT, XB1.VCC; no longer JP3.1, U$2.VCC, U1.AVCC, U1.VCC, U1.VCC_2
- net GND: now also J1.GND, J2.GND, SJ2.3, U$3.0
- net N$4: now also JP7.2; no longer JP1.1
- net N$5: now also JP8.2, U1.PD1_(TXD/PCINT17); no longer JP1.2, XB1.DOUT
- net N$6: now also J1.RXI, JP7.1; no longer JP2.1, XB1.DIN/!CONFIG
- net N$7: now also J1.TXO, JP8.1; no longer JP2.2, U1.PD1_(TXD/PCINT17)
Other:
- note added: "3V3: Direct 3.3v from XP Power +5V: 5V from RS232 connector VCC: Devices that use 3V3 or +5V"
- note added: "Connector is for one time usage only: Programming of Arduino bootloader. Connected directly to supply ATMEGA"
- moved on the sheet: JP4, JP5, R1, XB1

Commit message: 
Parts:
- removed JP1, JP8: (no value), jumper:JP2E
- added R4, R5, R6, R7: 4k7, rcl:R-EU_R0805
- IC1: value DS18B20 -> DS1820; device 1wire:DS18B20 -> DS1820:DS1820
- renumbered U$3 to PWR1
Connections:
- removed net +5V: J1.VCC, JP1.1
- removed net 1W: R1.1, U1.PD2_(INT0/PCINT18)
- removed net N$19: JP8.3, XB1.DIN/!CONFIG
- removed net N$7: J1.TXO, JP8.1
- new net N$6: IC1.DQ, R1.1, U1.PD2_(INT0/PCINT18)
- net +3V3: now also IC1.VDD, R4.2, R5.2; no longer JP1.3
- net GND: now also IC1.GND
- net N$10: now also R6.2, R7.2
- net N$12: now also R6.1
- net N$13: now also R7.1
- net N$5: now also J1.TXO, XB1.DIN/!CONFIG; no longer JP8.2
- net N$8: now also R4.1
- net N$9: now also R5.1
- net VCC: no longer JP1.2
Other:
- note added: "TxD and RxD are point of view from this device"
- note removed: "3V3: Direct 3.3v from XP Power +5V: 5V from RS232 connector VCC: Devices that use 3V3 or +5V"
- moved on the sheet: J1, JP4, JP5, X1

Commit message: base board
Parts:
- removed PWR1: IE0503D, xp_power:IE0503D
- added C10, C4, C5, C6, C7, C8, C9: 100n, rcl:C-EUC0805
- added C11: 10n, rcl:C-EUC0805
- added D1: RB161M-20TR, Components:RB161M-20TR
- added D2: BAT54HT1G, Components:BAT54HT1G
- added L1: VLCF4020, Components:VLCF4020
- added R10, R11, R13, R9: 4k7, rcl:R-EU_R0805
- added R8: 10k, rcl:R-EU_R0805
- added U$1: LM2736X, Components:LM2736X
- added U$3: XC6210, Components:XC6210
- U$2: value OLED_0.96_I2C -> OLED_0.96_I2CSWITCHPOWER; device tft_1.8_1.44_oled_0.96:OLED_0.96_I2C -> tft_1.8_1.44_oled_0.96:OLED_0.96_I2CSWITCHPOWER
Connections:
- removed net VCC: J2.CTS, LED1.A, SJ2.1, U$2.VCC, U1.AVCC, U1.VCC, U1.VCC_2
- new net N$19: C4.2, D2.C, U$1.BOOST
- new net N$25: R8.1, U$1.EN
- new net N$26: C9.2, IC1.VDD, R11.1
- new net N$27: C10.2, IC1.DQ, R13.1
- new net N$29: C11.2, U$3.NC
- new net VIN: JP6.2, R8.2, U$1.VIN
- new net VO: C5.2, D2.A, L1.2, R9.2, U$3.EN, U$3.IN
- net +3V3: now also C6.2, C7.2, C8.2, J2.CTS, LED1.A, R11.2, SJ2.1, U$2.VCC, U$3.OUT, U1.AVCC, U1.VCC, U1.VCC_2; no longer IC1.VDD, PWR1.+VOUT
- net GND: now also C10.1, C11.1, C5.1, C6.1, C7.1, C8.1, C9.1, D1.A, JP6.1, R10.1, U$1.GND, U$3.GND; no longer PWR1.0
- net N$11: now also C4.1, D1.C, L1.1, U$1.SW; no longer JP6.2, PWR1.+VIN
- net N$14: now also R10.2, R9.1, U$1.FB; no longer JP6.1, PWR1.-VIN
- net N$6: now also R13.2; no longer IC1.DQ
Other:
- moved on the sheet: JP6, R4, R5

Commit message: Voor aanpassing board (verplaatsen toetsen en xbee)
Parts:
- removed JP4: (no value), jumper:JP1E
- added C12: 1u, rcl:C-EUC0805
- R10: value 4k7 -> 21K5
- R11, R13: value 4k7 -> 560
- R6, R7: value 4k7 -> 1M
- R9: value 4k7 -> 10K
Connections:
- net +3V3: now also C12.2
- net GND: now also C12.1
- net N$10: no longer JP4.1, JP5.1
- net N$12: now also JP5.1; no longer JP4.2
Changed lines of the file:
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@@
 <part name="R1" library="rcl" deviceset="R-EU_" device="R0805" value="4k7"/>
 <part name="+3V5" library="supply1" deviceset="+3V3" device=""/>
-<part name="JP4" library="jumper" deviceset="JP1E" device=""/>
 <part name="JP5" library="jumper" deviceset="JP1E" device=""/>
 <part name="JP6" library="jumper" deviceset="JP1E" device=""/>
@@
 <part name="R5" library="rcl" deviceset="R-EU_" device="R0805" value="4k7"/>
 <part name="+3V1" library="supply1" deviceset="+3V3" device=""/>
-<part name="R6" library="rcl" deviceset="R-EU_" device="R0805" value="4k7"/>
-<part name="R7" library="rcl" deviceset="R-EU_" device="R0805" value="4k7"/>
+<part name="R6" library="rcl" deviceset="R-EU_" device="R0805" value="1M"/>
+<part name="R7" library="rcl" deviceset="R-EU_" device="R0805" value="1M"/>
 <part name="IC1" library="DS1820" deviceset="DS1820" device=""/>
 <part name="GND9" library="supply1" deviceset="GND" device=""/>
@@
 <part name="GND11" library="supply1" deviceset="GND" device=""/>
 <part name="C8" library="rcl" deviceset="C-EU" device="C0805" value="100n"/>
-<part name="R9" library="rcl" deviceset="R-EU_" device="R0805" value="4k7"/>
-<part name="R10" library="rcl" deviceset="R-EU_" device="R0805" value="4k7"/>
+<part name="R9" library="rcl" deviceset="R-EU_" device="R0805" value="10K"/>
+<part name="R10" library="rcl" deviceset="R-EU_" device="R0805" value="21K5"/>
 <part name="L1" library="Components" deviceset="VLCF4020" device=""/>
 <part name="D1" library="Components" deviceset="RB161M-20TR" device=""/>
@@
 <part name="GND12" library="supply1" deviceset="GND" device=""/>
 <part name="C9" library="rcl" deviceset="C-EU" device="C0805" value="100n"/>
-<part name="R11" library="rcl" deviceset="R-EU_" device="R0805" value="4k7"/>
+<part name="R11" library="rcl" deviceset="R-EU_" device="R0805" value="560"/>
 <part name="C10" library="rcl" deviceset="C-EU" device="C0805" value="100n"/>
-<part name="R13" library="rcl" deviceset="R-EU_" device="R0805" value="4k7"/>
+<part name="R13" library="rcl" deviceset="R-EU_" device="R0805" value="560"/>
 <part name="U$3" library="Components" deviceset="XC6210" device=""/>
 <part name="P+1" library="supply1" deviceset="+3V3" device=""/>
 <part name="C11" library="rcl" deviceset="C-EU" device="C0805" value="10n"/>
+<part name="C12" library="rcl" deviceset="C-EU" device="C0805" value="1u"/>
 </parts>
 <sheets>
@@
 <instance part="R1" gate="G$1" x="144.78" y="76.2" rot="R90"/>
 <instance part="+3V5" gate="G$1" x="144.78" y="86.36"/>
-<instance part="JP4" gate="A" x="165.1" y="58.42" rot="R270"/>
 <instance part="JP5" gate="A" x="172.72" y="55.88" rot="R270"/>
 <instance part="JP6" gate="A" x="-101.6" y="116.84" rot="R90"/>
@@
 </instance>
 <instance part="U$3" gate="G$1" x="27.94" y="109.22"/>
-<instance part="P+1" gate="G$1" x="53.34" y="121.92"/>
+<instance part="P+1" gate="G$1" x="60.96" y="121.92"/>
 <instance part="C11" gate="G$1" x="45.72" y="93.98" smashed="yes" rot="MR180">
 <attribute name="NAME" x="39.624" y="96.139" size="1.778" layer="95" rot="MR180"/>
 <attribute name="VALUE" x="49.784" y="96.139" size="1.778" layer="96" rot="MR180"/>
+</instance>
+<instance part="C12" gate="G$1" x="55.88" y="104.14" smashed="yes" rot="MR180">
+<attribute name="NAME" x="49.784" y="106.299" size="1.778" layer="95" rot="MR180"/>
+<attribute name="VALUE" x="59.944" y="106.299" size="1.778" layer="96" rot="MR180"/>
 </instance>
 </instances>
@@
 <wire x1="-15.24" y1="93.98" x2="-15.24" y2="91.44" width="0.1524" layer="91"/>
 <junction x="-15.24" y="91.44"/>
+<pinref part="C12" gate="G$1" pin="1"/>
+<wire x1="45.72" y1="91.44" x2="55.88" y2="91.44" width="0.1524" layer="91"/>
+<wire x1="55.88" y1="91.44" x2="55.88" y2="101.6" width="0.1524" layer="91"/>
+<junction x="45.72" y="91.44"/>
 </segment>
 <segment>
@@
 <segment>
 <pinref part="P+1" gate="G$1" pin="+3V3"/>
-<wire x1="53.34" y1="119.38" x2="53.34" y2="116.84" width="0.1524" layer="91"/>
+<wire x1="60.96" y1="119.38" x2="60.96" y2="116.84" width="0.1524" layer="91"/>
 <pinref part="U$3" gate="G$1" pin="OUT"/>
-<wire x1="53.34" y1="116.84" x2="45.72" y2="116.84" width="0.1524" layer="91"/>
+<wire x1="60.96" y1="116.84" x2="55.88" y2="116.84" width="0.1524" layer="91"/>
+<pinref part="C12" gate="G$1" pin="2"/>
+<wire x1="55.88" y1="116.84" x2="45.72" y2="116.84" width="0.1524" layer="91"/>
+<wire x1="55.88" y1="109.22" x2="55.88" y2="116.84" width="0.1524" layer="91"/>
+<junction x="55.88" y="116.84"/>
 </segment>
 </net>
@@
 <net name="N$10" class="0">
 <segment>
-<pinref part="JP4" gate="A" pin="1"/>
-<pinref part="U1" gate="A" pin="(PCINT19/OC2B/INT1)_PD3"/>
-<wire x1="162.56" y1="58.42" x2="142.24" y2="58.42" width="0.1524" layer="91"/>
-<wire x1="162.56" y1="58.42" x2="162.56" y2="60.96" width="0.1524" layer="91"/>
-<pinref part="JP5" gate="A" pin="1"/>
-<wire x1="162.56" y1="60.96" x2="170.18" y2="60.96" width="0.1524" layer="91"/>
-<wire x1="170.18" y1="60.96" x2="170.18" y2="55.88" width="0.1524" layer="91"/>
-<junction x="162.56" y="58.42"/>
 <pinref part="R6" gate="G$1" pin="2"/>
 <pinref part="R7" gate="G$1" pin="2"/>
 <wire x1="154.94" y1="81.28" x2="160.02" y2="81.28" width="0.1524" layer="91"/>
-<wire x1="160.02" y1="81.28" x2="170.18" y2="81.28" width="0.1524" layer="91"/>
-<wire x1="170.18" y1="81.28" x2="170.18" y2="60.96" width="0.1524" layer="91"/>
+<wire x1="160.02" y1="81.28" x2="165.1" y2="81.28" width="0.1524" layer="91"/>
+<wire x1="165.1" y1="81.28" x2="165.1" y2="58.42" width="0.1524" layer="91"/>
 <junction x="160.02" y="81.28"/>
-<junction x="170.18" y="60.96"/>
+<pinref part="U1" gate="A" pin="(PCINT19/OC2B/INT1)_PD3"/>
+<wire x1="162.56" y1="58.42" x2="142.24" y2="58.42" width="0.1524" layer="91"/>
+<wire x1="165.1" y1="58.42" x2="162.56" y2="58.42" width="0.1524" layer="91"/>
 </segment>
 </net>
@@
 <segment>
 <pinref part="U1" gate="A" pin="(PCINT20/XCK/T0)_PD4"/>
-<pinref part="JP4" gate="A" pin="2"/>
 <wire x1="142.24" y1="55.88" x2="154.94" y2="55.88" width="0.1524" layer="91"/>
 <pinref part="R6" gate="G$1" pin="1"/>
-<wire x1="154.94" y1="55.88" x2="162.56" y2="55.88" width="0.1524" layer="91"/>
 <wire x1="154.94" y1="71.12" x2="154.94" y2="55.88" width="0.1524" layer="91"/>
+<pinref part="JP5" gate="A" pin="1"/>
+<wire x1="154.94" y1="55.88" x2="170.18" y2="55.88" width="0.1524" layer="91"/>
 <junction x="154.94" y="55.88"/>
 </segment>

Commit message: power routed/ labels placed
Parts:
- renumbered U$1 to U2, U$3 to U3
Changed lines of the file:
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@@
 <part name="GND9" library="supply1" deviceset="GND" device=""/>
 <part name="+3V2" library="supply1" deviceset="+3V3" device=""/>
-<part name="U$1" library="Components" deviceset="LM2736X" device=""/>
+<part name="U2" library="Components" deviceset="LM2736X" device=""/>
 <part name="R8" library="rcl" deviceset="R-EU_" device="R0805" value="10k"/>
 <part name="C4" library="rcl" deviceset="C-EU" device="C0805" value="100n"/>
@@
 <part name="C10" library="rcl" deviceset="C-EU" device="C0805" value="100n"/>
 <part name="R13" library="rcl" deviceset="R-EU_" device="R0805" value="560"/>
-<part name="U$3" library="Components" deviceset="XC6210" device=""/>
+<part name="U3" library="Components" deviceset="XC6210" device=""/>
 <part name="P+1" library="supply1" deviceset="+3V3" device=""/>
 <part name="C11" library="rcl" deviceset="C-EU" device="C0805" value="10n"/>
@@
 <instance part="GND9" gate="1" x="165.1" y="10.16"/>
 <instance part="+3V2" gate="G$1" x="142.24" y="27.94"/>
-<instance part="U$1" gate="G$1" x="-58.42" y="116.84"/>
+<instance part="U2" gate="G$1" x="-58.42" y="116.84"/>
 <instance part="R8" gate="G$1" x="-76.2" y="116.84" rot="R90"/>
 <instance part="C4" gate="G$1" x="-40.64" y="119.38" smashed="yes" rot="MR180">
@@
 <attribute name="VALUE" x="181.102" y="24.13" size="1.778" layer="96" rot="R90"/>
 </instance>
-<instance part="U$3" gate="G$1" x="27.94" y="109.22"/>
+<instance part="U3" gate="G$1" x="27.94" y="109.22"/>
 <instance part="P+1" gate="G$1" x="60.96" y="121.92"/>
 <instance part="C11" gate="G$1" x="45.72" y="93.98" smashed="yes" rot="MR180">
@@
 </segment>
 <segment>
-<pinref part="U$1" gate="G$1" pin="GND"/>
+<pinref part="U2" gate="G$1" pin="GND"/>
 <pinref part="GND5" gate="1" pin="GND"/>
 <wire x1="-60.96" y1="96.52" x2="-60.96" y2="91.44" width="0.1524" layer="91"/>
@@
 <wire x1="-27.94" y1="91.44" x2="-35.56" y2="91.44" width="0.1524" layer="91"/>
 <wire x1="-35.56" y1="91.44" x2="-40.64" y2="91.44" width="0.1524" layer="91"/>
-<pinref part="U$3" gate="G$1" pin="GND"/>
+<pinref part="U3" gate="G$1" pin="GND"/>
 <wire x1="-40.64" y1="91.44" x2="-60.96" y2="91.44" width="0.1524" layer="91"/>
 <wire x1="-7.62" y1="91.44" x2="30.48" y2="91.44" width="0.1524" layer="91"/>
@@
 <pinref part="P+1" gate="G$1" pin="+3V3"/>
 <wire x1="60.96" y1="119.38" x2="60.96" y2="116.84" width="0.1524" layer="91"/>
-<pinref part="U$3" gate="G$1" pin="OUT"/>
+<pinref part="U3" gate="G$1" pin="OUT"/>
 <wire x1="60.96" y1="116.84" x2="55.88" y2="116.84" width="0.1524" layer="91"/>
 <pinref part="C12" gate="G$1" pin="2"/>
@@
 <wire x1="-99.06" y1="119.38" x2="-93.98" y2="119.38" width="0.1524" layer="91"/>
 <wire x1="-93.98" y1="119.38" x2="-93.98" y2="124.46" width="0.1524" layer="91"/>
-<pinref part="U$1" gate="G$1" pin="VIN"/>
+<pinref part="U2" gate="G$1" pin="VIN"/>
 <wire x1="-93.98" y1="124.46" x2="-76.2" y2="124.46" width="0.1524" layer="91"/>
 <pinref part="R8" gate="G$1" pin="2"/>
@@
 <net name="N$19" class="1">
 <segment>
-<pinref part="U$1" gate="G$1" pin="BOOST"/>
+<pinref part="U2" gate="G$1" pin="BOOST"/>
 <pinref part="C4" gate="G$1" pin="2"/>
 <wire x1="-45.72" y1="124.46" x2="-40.64" y2="124.46" width="0.1524" layer="91"/>
@@
 <pinref part="R8" gate="G$1" pin="1"/>
 <wire x1="-76.2" y1="111.76" x2="-76.2" y2="106.68" width="0.1524" layer="91"/>
-<pinref part="U$1" gate="G$1" pin="EN"/>
+<pinref part="U2" gate="G$1" pin="EN"/>
 <wire x1="-76.2" y1="106.68" x2="-73.66" y2="106.68" width="0.1524" layer="91"/>
 </segment>
@@
 <wire x1="-7.62" y1="132.08" x2="-7.62" y2="116.84" width="0.1524" layer="91"/>
 <junction x="-7.62" y="116.84"/>
-<pinref part="U$3" gate="G$1" pin="IN"/>
+<pinref part="U3" gate="G$1" pin="IN"/>
 <wire x1="-7.62" y1="116.84" x2="15.24" y2="116.84" width="0.1524" layer="91"/>
-<pinref part="U$3" gate="G$1" pin="EN"/>
+<pinref part="U3" gate="G$1" pin="EN"/>
 <wire x1="15.24" y1="116.84" x2="15.24" y2="104.14" width="0.1524" layer="91"/>
 <junction x="15.24" y="116.84"/>
@@
 <net name="N$29" class="0">
 <segment>
-<pinref part="U$3" gate="G$1" pin="NC"/>
+<pinref part="U3" gate="G$1" pin="NC"/>
 <pinref part="C11" gate="G$1" pin="2"/>
 <wire x1="45.72" y1="104.14" x2="45.72" y2="99.06" width="0.1524" layer="91"/>
@@
 <segment>
 <pinref part="C4" gate="G$1" pin="1"/>
-<pinref part="U$1" gate="G$1" pin="SW"/>
+<pinref part="U2" gate="G$1" pin="SW"/>
 <wire x1="-45.72" y1="116.84" x2="-40.64" y2="116.84" width="0.1524" layer="91"/>
 <pinref part="L1" gate="G$1" pin="1"/>
@@
 <pinref part="R9" gate="G$1" pin="1"/>
 <pinref part="R10" gate="G$1" pin="2"/>
-<pinref part="U$1" gate="G$1" pin="FB"/>
+<pinref part="U2" gate="G$1" pin="FB"/>
 <wire x1="-45.72" y1="106.68" x2="-25.4" y2="106.68" width="0.1524" layer="91"/>
 <wire x1="-25.4" y1="106.68" x2="-25.4" y2="104.14" width="0.1524" layer="91"/>

Commit message: input cap toegevoegd
Parts:
- added C13: 10u, rcl:C-EUC0805
Connections:
- net GND: now also C13.1
- net VIN: now also C13.2
Changed lines of the file:
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@@
 <part name="C11" library="rcl" deviceset="C-EU" device="C0805" value="10n"/>
 <part name="C12" library="rcl" deviceset="C-EU" device="C0805" value="1u"/>
+<part name="C13" library="rcl" deviceset="C-EU" device="C0805" value="10u"/>
 </parts>
 <sheets>
@@
 <attribute name="VALUE" x="59.944" y="106.299" size="1.778" layer="96" rot="MR180"/>
 </instance>
+<instance part="C13" gate="G$1" x="-88.9" y="104.14" rot="MR180"/>
 </instances>
 <busses>
@@
 <wire x1="-99.06" y1="116.84" x2="-93.98" y2="116.84" width="0.1524" layer="91"/>
 <wire x1="-93.98" y1="116.84" x2="-93.98" y2="91.44" width="0.1524" layer="91"/>
-<wire x1="-93.98" y1="91.44" x2="-60.96" y2="91.44" width="0.1524" layer="91"/>
+<wire x1="-93.98" y1="91.44" x2="-88.9" y2="91.44" width="0.1524" layer="91"/>
 <junction x="-60.96" y="91.44"/>
 <pinref part="C5" gate="G$1" pin="1"/>
+<wire x1="-88.9" y1="91.44" x2="-60.96" y2="91.44" width="0.1524" layer="91"/>
 <wire x1="-7.62" y1="106.68" x2="-7.62" y2="91.44" width="0.1524" layer="91"/>
 <wire x1="-7.62" y1="91.44" x2="-15.24" y2="91.44" width="0.1524" layer="91"/>
@@
 <wire x1="55.88" y1="91.44" x2="55.88" y2="101.6" width="0.1524" layer="91"/>
 <junction x="45.72" y="91.44"/>
+<pinref part="C13" gate="G$1" pin="1"/>
+<wire x1="-88.9" y1="101.6" x2="-88.9" y2="91.44" width="0.1524" layer="91"/>
+<junction x="-88.9" y="91.44"/>
 </segment>
 <segment>
@@
 <wire x1="-93.98" y1="119.38" x2="-93.98" y2="124.46" width="0.1524" layer="91"/>
 <pinref part="U2" gate="G$1" pin="VIN"/>
-<wire x1="-93.98" y1="124.46" x2="-76.2" y2="124.46" width="0.1524" layer="91"/>
+<wire x1="-93.98" y1="124.46" x2="-88.9" y2="124.46" width="0.1524" layer="91"/>
 <pinref part="R8" gate="G$1" pin="2"/>
+<wire x1="-88.9" y1="124.46" x2="-76.2" y2="124.46" width="0.1524" layer="91"/>
 <wire x1="-76.2" y1="124.46" x2="-73.66" y2="124.46" width="0.1524" layer="91"/>
 <wire x1="-76.2" y1="124.46" x2="-76.2" y2="121.92" width="0.1524" layer="91"/>
 <junction x="-76.2" y="124.46"/>
-</segment>
-</net>
+<pinref part="C13" gate="G$1" pin="2"/>
+<wire x1="-88.9" y1="109.22" x2="-88.9" y2="124.46" width="0.1524" layer="91"/>
+<junction x="-88.9" y="124.46"/>
+</segment>
+</net>

Commit message: 
Connections:
- net N$8 renamed SDA
- net N$9 renamed SCL
Changed lines of the file:
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@@
 </segment>
 </net>
-<net name="N$8" class="0">
+<net name="SDA" class="0">
 <segment>
 <pinref part="U$2" gate="G$1" pin="SDA"/>
@@
 </segment>
 </net>
-<net name="N$9" class="0">
+<net name="SCL" class="0">
 <segment>
 <pinref part="U$2" gate="G$1" pin="SCL"/>

Commit message: component values
Parts:
- C5: value 100n -> 10u
- R11, R13: value 560 -> 580
Changed lines of the file:
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@@
 <part name="R8" library="rcl" deviceset="R-EU_" device="R0805" value="10k"/>
 <part name="C4" library="rcl" deviceset="C-EU" device="C0805" value="100n"/>
-<part name="C5" library="rcl" deviceset="C-EU" device="C0805" value="100n"/>
+<part name="C5" library="rcl" deviceset="C-EU" device="C0805" value="10u"/>
 <part name="C6" library="rcl" deviceset="C-EU" device="C0805" value="100n"/>
 <part name="GND10" library="supply1" deviceset="GND" device=""/>
@@
 <part name="GND12" library="supply1" deviceset="GND" device=""/>
 <part name="C9" library="rcl" deviceset="C-EU" device="C0805" value="100n"/>
-<part name="R11" library="rcl" deviceset="R-EU_" device="R0805" value="560"/>
+<part name="R11" library="rcl" deviceset="R-EU_" device="R0805" value="580"/>
 <part name="C10" library="rcl" deviceset="C-EU" device="C0805" value="100n"/>
-<part name="R13" library="rcl" deviceset="R-EU_" device="R0805" value="560"/>
+<part name="R13" library="rcl" deviceset="R-EU_" device="R0805" value="580"/>
 <part name="U3" library="Components" deviceset="XC6210" device=""/>
 <part name="P+1" library="supply1" deviceset="+3V3" device=""/>
