File: Arduino/PCB/TempSensor/TempSensor.sch (EAGLE design)
At the start: 42 parts, among them IC1 DS1820, J1 FTDI_DEVICE, J2 FTDI_DEVICE, U1 ATMEGA328-AU, U2 LM2736X, U3 XC6210, X1 16Mhz

Commit message: part values
Parts:
- C10, C9: value 100n -> 220p
- R10: value 21K5 -> 10K
- R11, R13: value 580 -> 100
- R9: value 10K -> 21K5
Changed lines of the file:
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@@
 <part name="GND11" library="supply1" deviceset="GND" device=""/>
 <part name="C8" library="rcl" deviceset="C-EU" device="C0805" value="100n"/>
-<part name="R9" library="rcl" deviceset="R-EU_" device="R0805" value="10K"/>
-<part name="R10" library="rcl" deviceset="R-EU_" device="R0805" value="21K5"/>
+<part name="R9" library="rcl" deviceset="R-EU_" device="R0805" value="21K5"/>
+<part name="R10" library="rcl" deviceset="R-EU_" device="R0805" value="10K"/>
 <part name="L1" library="Components" deviceset="VLCF4020" device=""/>
 <part name="D1" library="Components" deviceset="RB161M-20TR" device=""/>
 <part name="D2" library="Components" deviceset="BAT54HT1G" device=""/>
 <part name="GND12" library="supply1" deviceset="GND" device=""/>
-<part name="C9" library="rcl" deviceset="C-EU" device="C0805" value="100n"/>
-<part name="R11" library="rcl" deviceset="R-EU_" device="R0805" value="580"/>
-<part name="C10" library="rcl" deviceset="C-EU" device="C0805" value="100n"/>
-<part name="R13" library="rcl" deviceset="R-EU_" device="R0805" value="580"/>
+<part name="C9" library="rcl" deviceset="C-EU" device="C0805" value="220p"/>
+<part name="R11" library="rcl" deviceset="R-EU_" device="R0805" value="100"/>
+<part name="C10" library="rcl" deviceset="C-EU" device="C0805" value="220p"/>
+<part name="R13" library="rcl" deviceset="R-EU_" device="R0805" value="100"/>
 <part name="U3" library="Components" deviceset="XC6210" device=""/>
 <part name="P+1" library="supply1" deviceset="+3V3" device=""/>
