File: Arduino/PCB/MainBoard/Mainboard.sch (EAGLE design)
At the start: 62 parts, among them IC1 ULN2803ADW, IC2 DS1338Z-33+, J1 ARDUINO PROG, J2 BOOTL PROG, J3 DC-005, J4 XBEE CONN, Q1 32.768kHz, U1 ATMEGA328-AU, U4 R-78B5.0-2.0, X1 16Mhz

Commit message: ready to send v2
Connections:
- net GND: now also JP1.14, JP1.20, JP1.6, JP1.9
- net N$15: now also X3-2.KL; no longer X3-1.KL
- net N$16: now also X3-3.KL; no longer X3-4.KL
- net N$17: now also X3-4.KL; no longer X3-3.KL
- net N$18: now also X3-5.KL; no longer X3-6.KL
- net N$19: now also X3-6.KL; no longer X3-5.KL
- net N$21: now also X3-7.KL; no longer X3-8.KL
- net N$23: now also X4-7.KL; no longer X4-8.KL
- net N$25: now also X3-8.KL; no longer X3-7.KL
- net N$26: now also X4-1.KL; no longer X4-2.KL
- net N$27: now also X4-2.KL; no longer X4-1.KL
- net N$28: now also X4-3.KL; no longer X4-4.KL
- net N$29: now also X4-4.KL; no longer X4-3.KL
- net N$30: now also X4-5.KL; no longer X4-6.KL
- net N$31: now also X4-6.KL; no longer X4-5.KL
- net N$33: now also X4-8.KL; no longer X4-7.KL
- net N$4: now also X3-1.KL; no longer X3-2.KL
Other:
- moved on the sheet: X3-1, X3-2, X3-3, X3-4, X3-5, X3-6, X3-7, X3-8, X4-1, X4-2, X4-3, X4-4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
Changed lines of the file:
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@@
 <part name="LED10" library="led" deviceset="LED" device="3MM" value="2mA"/>
 <part name="U$1" library="MainboardComponents" deviceset="KEYSTONE_1066" device=""/>
+<part name="GND7" library="supply1" deviceset="GND" device=""/>
+<part name="GND18" library="supply1" deviceset="GND" device=""/>
+<part name="GND19" library="supply1" deviceset="GND" device=""/>
+<part name="GND20" library="supply1" deviceset="GND" device=""/>
 </parts>
 <sheets>
@@
 <attribute name="VALUE" x="271.78" y="-81.28" size="1.778" layer="94"/>
 </instance>
-<instance part="X3" gate="-1" x="309.88" y="40.64" rot="R180"/>
-<instance part="X3" gate="-2" x="309.88" y="45.72" rot="R180"/>
-<instance part="X3" gate="-3" x="309.88" y="30.48" rot="R180"/>
-<instance part="X3" gate="-4" x="309.88" y="35.56" rot="R180"/>
-<instance part="X3" gate="-5" x="309.88" y="20.32" rot="R180"/>
-<instance part="X3" gate="-6" x="309.88" y="25.4" rot="R180"/>
-<instance part="X3" gate="-7" x="309.88" y="10.16" rot="R180"/>
-<instance part="X3" gate="-8" x="309.88" y="15.24" rot="R180"/>
-<instance part="X4" gate="-1" x="309.88" y="-20.32" rot="R180"/>
-<instance part="X4" gate="-2" x="309.88" y="-15.24" rot="R180"/>
-<instance part="X4" gate="-3" x="309.88" y="-30.48" rot="R180"/>
-<instance part="X4" gate="-4" x="309.88" y="-25.4" rot="R180"/>
-<instance part="X4" gate="-5" x="309.88" y="-40.64" rot="R180"/>
-<instance part="X4" gate="-6" x="309.88" y="-35.56" rot="R180"/>
-<instance part="X4" gate="-7" x="309.88" y="-50.8" rot="R180"/>
-<instance part="X4" gate="-8" x="309.88" y="-45.72" rot="R180"/>
+<instance part="X3" gate="-1" x="309.88" y="45.72" rot="R180"/>
+<instance part="X3" gate="-2" x="309.88" y="40.64" rot="R180"/>
+<instance part="X3" gate="-3" x="309.88" y="35.56" rot="R180"/>
+<instance part="X3" gate="-4" x="309.88" y="30.48" rot="R180"/>
+<instance part="X3" gate="-5" x="309.88" y="25.4" rot="R180"/>
+<instance part="X3" gate="-6" x="309.88" y="20.32" rot="R180"/>
+<instance part="X3" gate="-7" x="309.88" y="15.24" rot="R180"/>
+<instance part="X3" gate="-8" x="309.88" y="10.16" rot="R180"/>
+<instance part="X4" gate="-1" x="309.88" y="-15.24" rot="R180"/>
+<instance part="X4" gate="-2" x="309.88" y="-20.32" rot="R180"/>
+<instance part="X4" gate="-3" x="309.88" y="-25.4" rot="R180"/>
+<instance part="X4" gate="-4" x="309.88" y="-30.48" rot="R180"/>
+<instance part="X4" gate="-5" x="309.88" y="-35.56" rot="R180"/>
+<instance part="X4" gate="-6" x="309.88" y="-40.64" rot="R180"/>
+<instance part="X4" gate="-7" x="309.88" y="-45.72" rot="R180"/>
+<instance part="X4" gate="-8" x="309.88" y="-50.8" rot="R180"/>
 <instance part="JP2" gate="A" x="-33.02" y="76.2" rot="R90"/>
 <instance part="GND12" gate="1" x="-27.94" y="71.12"/>
@@
 <attribute name="VALUE" x="-144.78" y="-22.86" size="1.778" layer="96" rot="R90"/>
 </instance>
+<instance part="GND7" gate="1" x="-149.86" y="12.7"/>
+<instance part="GND18" gate="1" x="-195.58" y="7.62"/>
+<instance part="GND19" gate="1" x="-162.56" y="2.54"/>
+<instance part="GND20" gate="1" x="-162.56" y="-7.62"/>
 </instances>
 <busses>
@@
 <pinref part="U$1" gate="G$1" pin="-"/>
 <wire x1="-139.7" y1="-22.86" x2="-139.7" y2="-20.32" width="0.1524" layer="91"/>
+</segment>
+<segment>
+<pinref part="JP1" gate="A" pin="6"/>
+<pinref part="GND7" gate="1" pin="GND"/>
+<wire x1="-170.18" y1="15.24" x2="-149.86" y2="15.24" width="0.1524" layer="91"/>
+</segment>
+<segment>
+<pinref part="JP1" gate="A" pin="9"/>
+<pinref part="GND18" gate="1" pin="GND"/>
+<wire x1="-177.8" y1="10.16" x2="-195.58" y2="10.16" width="0.1524" layer="91"/>
+</segment>
+<segment>
+<pinref part="JP1" gate="A" pin="14"/>
+<pinref part="GND19" gate="1" pin="GND"/>
+<wire x1="-170.18" y1="5.08" x2="-162.56" y2="5.08" width="0.1524" layer="91"/>
+</segment>
+<segment>
+<pinref part="JP1" gate="A" pin="20"/>
+<pinref part="GND20" gate="1" pin="GND"/>
+<wire x1="-170.18" y1="-2.54" x2="-162.56" y2="-2.54" width="0.1524" layer="91"/>
+<wire x1="-162.56" y1="-2.54" x2="-162.56" y2="-5.08" width="0.1524" layer="91"/>
 </segment>
 </net>
@@
 <wire x1="269.24" y1="68.58" x2="299.72" y2="68.58" width="0.1524" layer="91"/>
 <wire x1="299.72" y1="68.58" x2="299.72" y2="45.72" width="0.1524" layer="91"/>
-<pinref part="X3" gate="-2" pin="KL"/>
+<pinref part="X3" gate="-1" pin="KL"/>
 <wire x1="299.72" y1="45.72" x2="304.8" y2="45.72" width="0.1524" layer="91"/>
 </segment>
@@
 <wire x1="269.24" y1="53.34" x2="297.18" y2="53.34" width="0.1524" layer="91"/>
 <wire x1="297.18" y1="53.34" x2="297.18" y2="40.64" width="0.1524" layer="91"/>
-<pinref part="X3" gate="-1" pin="KL"/>
+<pinref part="X3" gate="-2" pin="KL"/>
 <wire x1="297.18" y1="40.64" x2="304.8" y2="40.64" width="0.1524" layer="91"/>
 </segment>
@@
 <wire x1="269.24" y1="48.26" x2="294.64" y2="48.26" width="0.1524" layer="91"/>
 <wire x1="294.64" y1="48.26" x2="294.64" y2="35.56" width="0.1524" layer="91"/>
-<pinref part="X3" gate="-4" pin="KL"/>
+<pinref part="X3" gate="-3" pin="KL"/>
 <wire x1="294.64" y1="35.56" x2="304.8" y2="35.56" width="0.1524" layer="91"/>
 </segment>
@@
 <pinref part="REL1" gate="G$1" pin="C"/>
 <wire x1="269.24" y1="33.02" x2="304.8" y2="33.02" width="0.1524" layer="91"/>
-<pinref part="X3" gate="-3" pin="KL"/>
+<pinref part="X3" gate="-4" pin="KL"/>
 <wire x1="304.8" y1="33.02" x2="304.8" y2="30.48" width="0.1524" layer="91"/>
 </segment>
@@
 <wire x1="269.24" y1="12.7" x2="289.56" y2="12.7" width="0.1524" layer="91"/>
 <wire x1="289.56" y1="12.7" x2="289.56" y2="20.32" width="0.1524" layer="91"/>
-<pinref part="X3" gate="-5" pin="KL"/>
+<pinref part="X3" gate="-6" pin="KL"/>
 <wire x1="289.56" y1="20.32" x2="304.8" y2="20.32" width="0.1524" layer="91"/>
 </segment>
@@
 <wire x1="269.24" y1="7.62" x2="292.1" y2="7.62" width="0.1524" layer="91"/>
 <wire x1="292.1" y1="7.62" x2="292.1" y2="15.24" width="0.1524" layer="91"/>
-<pinref part="X3" gate="-8" pin="KL"/>
+<pinref part="X3" gate="-7" pin="KL"/>
 <wire x1="292.1" y1="15.24" x2="304.8" y2="15.24" width="0.1524" layer="91"/>
 </segment>
@@
 <wire x1="269.24" y1="-7.62" x2="299.72" y2="-7.62" width="0.1524" layer="91"/>
 <wire x1="299.72" y1="-7.62" x2="299.72" y2="10.16" width="0.1524" layer="91"/>
-<pinref part="X3" gate="-7" pin="KL"/>
+<pinref part="X3" gate="-8" pin="KL"/>
 <wire x1="299.72" y1="10.16" x2="304.8" y2="10.16" width="0.1524" layer="91"/>
 </segment>
@@
 <wire x1="269.24" y1="-27.94" x2="289.56" y2="-27.94" width="0.1524" layer="91"/>
 <wire x1="289.56" y1="-27.94" x2="289.56" y2="-20.32" width="0.1524" layer="91"/>
-<pinref part="X4" gate="-1" pin="KL"/>
+<pinref part="X4" gate="-2" pin="KL"/>
 <wire x1="289.56" y1="-20.32" x2="304.8" y2="-20.32" width="0.1524" layer="91"/>
 </segment>
@@
 <wire x1="269.24" y1="-33.02" x2="292.1" y2="-33.02" width="0.1524" layer="91"/>
 <wire x1="292.1" y1="-33.02" x2="292.1" y2="-25.4" width="0.1524" layer="91"/>
-<pinref part="X4" gate="-4" pin="KL"/>
+<pinref part="X4" gate="-3" pin="KL"/>
 <wire x1="292.1" y1="-25.4" x2="304.8" y2="-25.4" width="0.1524" layer="91"/>
 </segment>
@@
 <wire x1="269.24" y1="-48.26" x2="294.64" y2="-48.26" width="0.1524" layer="91"/>
 <wire x1="294.64" y1="-48.26" x2="294.64" y2="-30.48" width="0.1524" layer="91"/>
-<pinref part="X4" gate="-3" pin="KL"/>
+<pinref part="X4" gate="-4" pin="KL"/>
 <wire x1="294.64" y1="-30.48" x2="304.8" y2="-30.48" width="0.1524" layer="91"/>
 </segment>
@@
 <wire x1="269.24" y1="-53.34" x2="297.18" y2="-53.34" width="0.1524" layer="91"/>
 <wire x1="297.18" y1="-53.34" x2="297.18" y2="-35.56" width="0.1524" layer="91"/>
-<pinref part="X4" gate="-6" pin="KL"/>
+<pinref part="X4" gate="-5" pin="KL"/>
 <wire x1="297.18" y1="-35.56" x2="304.8" y2="-35.56" width="0.1524" layer="91"/>
 </segment>
@@
 <wire x1="269.24" y1="-68.58" x2="299.72" y2="-68.58" width="0.1524" layer="91"/>
 <wire x1="299.72" y1="-68.58" x2="299.72" y2="-40.64" width="0.1524" layer="91"/>
-<pinref part="X4" gate="-5" pin="KL"/>
+<pinref part="X4" gate="-6" pin="KL"/>
 <wire x1="299.72" y1="-40.64" x2="304.8" y2="-40.64" width="0.1524" layer="91"/>
 </segment>
@@
 <pinref part="REL7" gate="G$1" pin="C"/>
 <wire x1="269.24" y1="-88.9" x2="304.8" y2="-88.9" width="0.1524" layer="91"/>
-<pinref part="X4" gate="-7" pin="KL"/>
+<pinref part="X4" gate="-8" pin="KL"/>
 <wire x1="304.8" y1="-88.9" x2="304.8" y2="-50.8" width="0.1524" layer="91"/>
 </segment>
@@
 <wire x1="269.24" y1="27.94" x2="302.26" y2="27.94" width="0.1524" layer="91"/>
 <wire x1="302.26" y1="27.94" x2="302.26" y2="25.4" width="0.1524" layer="91"/>
-<pinref part="X3" gate="-6" pin="KL"/>
+<pinref part="X3" gate="-5" pin="KL"/>
 <wire x1="302.26" y1="25.4" x2="304.8" y2="25.4" width="0.1524" layer="91"/>
 </segment>
@@
 <wire x1="269.24" y1="-12.7" x2="302.26" y2="-12.7" width="0.1524" layer="91"/>
 <wire x1="302.26" y1="-12.7" x2="302.26" y2="-15.24" width="0.1524" layer="91"/>
-<pinref part="X4" gate="-2" pin="KL"/>
+<pinref part="X4" gate="-1" pin="KL"/>
 <wire x1="302.26" y1="-15.24" x2="304.8" y2="-15.24" width="0.1524" layer="91"/>
 </segment>
@@
 <net name="N$23" class="2">
 <segment>
-<pinref part="X4" gate="-8" pin="KL"/>
-<wire x1="304.8" y1="-45.72" x2="302.26" y2="-45.72" width="0.1524" layer="91"/>
 <wire x1="302.26" y1="-45.72" x2="302.26" y2="-73.66" width="0.1524" layer="91"/>
 <pinref part="REL7" gate="G$1" pin="NO"/>
 <wire x1="302.26" y1="-73.66" x2="269.24" y2="-73.66" width="0.1524" layer="91"/>
-</segment>
-</net>
+<pinref part="X4" gate="-7" pin="KL"/>
+<wire x1="302.26" y1="-45.72" x2="304.8" y2="-45.72" width="0.1524" layer="91"/>
+</segment>
+</net>
